Commit message: [script_hpp/urdf/srdf] modifications of the pedestal position

File: urdf/support.urdf.xacro (robot description, xacro)
@@ -175,5 +175,5 @@
       </joint>
       <joint name="pedestal_joint" type="fixed">
-        <origin xyz="1.05 0.45 0"/>
+        <origin xyz="1.05 0 0"/>
         <parent link="world"/>
         <child link="pedestal"/>
