Commit message: Change camera support

File: urdf/franka_robot.xacro (robot description, xacro)
@@ -49,13 +49,13 @@
       </inertial>
       <visual>
-        <origin xyz="0.022 -0.102 -0.035" rpy="3.141592653589793 0 -1.5707963267948966"/>
+        <origin xyz="0.022 0 -0.012" rpy="3.141592653589793 0 -1.5707963267948966"/>
         <geometry>
-          <mesh filename="package://agimus_demos/franka/manipulation/meshes/camera-support.stl" scale="0.001 0.001 0.001"/>
+          <mesh filename="package://agimus_demos/franka/manipulation/meshes/camera-support.stl" scale="1 1 1"/>
         </geometry>
       </visual>
       <collision>
-        <origin xyz="0.022 -0.102 -0.035" rpy="3.141592653589793 0 -1.5707963267948966"/>
+        <origin xyz="0.022 0 -0.012" rpy="3.141592653589793 0 -1.5707963267948966"/>
         <geometry>
-          <mesh filename="package://agimus_demos/franka/manipulation/meshes/camera-support.stl" scale="0.001 0.001 0.001"/>
+          <mesh filename="package://agimus_demos/franka/manipulation/meshes/camera-support.stl" scale="1 1 1"/>
         </geometry>
       </collision>
